File: project.sch (EAGLE design)
At the start: 44 parts, among them IC1 UA78M33CDCYG3, U1 DSPIC33FJ64MC804-H/PT, U2 TB6612FNG,C,8,EL, Y1 ABM8-20.000MHZ-B2-T

Commit message: Renamed Components
Parts:
- C14: value 0.1uF -> 0.33µF
- C15: value 10µF -> 0.1µF
- renumbered IC1 to LINEAR_REGULATOR, JP2 to PROGRAMMER_PO, JP3 to DEBUGGING_PO, MOTOR_A to MOTOR_L, MOTOR_B to MOTOR_R, U1 to MICROCHIP, U2 to HBRIDGE, Y1 to OSC

Commit message: kleine Änderungen
Parts:
- removed JP1: (no value), pinhead:PINHD-1X2
- removed LINEAR_REGULATOR: UA78M33CDCYG3, UA78M33CDCYG3:UA78M33CDCYG3
- added BATTERY: (no value), pinhead:PINHD-1X2
- added LINEAR_REGULATOR_3.3V: UA78M33CDCYG3, UA78M33CDCYG3:UA78M33CDCYG3
Connections:
- net GND: now also BATTERY.2, LINEAR_REGULATOR_3.3V.COMMON_1, LINEAR_REGULATOR_3.3V.COMMON_2; no longer JP1.2, LINEAR_REGULATOR.COMMON_1, LINEAR_REGULATOR.COMMON_2
- net N$6: now also BATTERY.1, LINEAR_REGULATOR_3.3V.INPUT; no longer JP1.1, LINEAR_REGULATOR.INPUT
- net VCC: now also LINEAR_REGULATOR_3.3V.OUTPUT; no longer LINEAR_REGULATOR.OUTPUT
Other:
- moved on the sheet: BLUETOOTH_UART, C14, C15, C16, C17, DEBUGGING_PO, HBRIDGE, MOTOR_L

Commit message: Oscillator
Parts:
- removed OSC: ABM8-20.000MHZ-B2-T, ABM8-20.000MHZ-B2-T:ABM8-20.000MHZ-B2-T
- added Y1: ABM8-20.000MHZ-B2-T, ABM8-20.000MHZ-B2-T:ABM8-20.000MHZ-B2-T
Connections:
- removed net ENCA_B: MOTOR_L.6
- removed net N$6: BATTERY.1, C14.1, LINEAR_REGULATOR_3.3V.INPUT
- new net B01: HBRIDGE.BO1_2
- new net MTRDRV_AI1: HBRIDGE.AIN1
- new net N$4: C3.2, Y1.X2
- new net VM: BATTERY.1, C14.1, C8.1, C9.1, HBRIDGE.VM1, HBRIDGE.VM2, HBRIDGE.VM3, LINEAR_REGULATOR_3.3V.INPUT
- net AO1: now also HBRIDGE.AO1_1, HBRIDGE.AO1_2; no longer HBRIDGE.AO1@1, HBRIDGE.AO1@2
- net AO2: now also HBRIDGE.AO2_1, HBRIDGE.AO2_2; no longer HBRIDGE.AO2@1, HBRIDGE.AO2@2
- net BO1: no longer HBRIDGE.BO1@1, HBRIDGE.BO1@2
- net BO2: now also HBRIDGE.BO2_1, HBRIDGE.BO2_2; no longer HBRIDGE.BO2@1, HBRIDGE.BO2@2
- net ENCA_A: now also MOTOR_L.6
- net GND: now also HBRIDGE.PGND1_1, HBRIDGE.PGND1_2, HBRIDGE.PGND2_1, HBRIDGE.PGND2_2, Y1.GND_1, Y1.GND_2; no longer C2.1, C3.1, OSC.GND
- net MTRDRV_AIN1: no longer HBRIDGE.AIN1
- net N$1: now also C3.1; no longer C2.2, OSC.1
- net N$2: now also C2.2; no longer C3.2, OSC.2
- net N$3: now also C2.1, Y1.X1; no longer C8.1, C9.1, HBRIDGE.VM1, HBRIDGE.VM2, HBRIDGE.VM3
Other:
- moved on the sheet: C2, C3, C8, C9, HBRIDGE

Commit message: Kleine Änderungen
Connections:
- removed net N$9: D1.A, R4.2
- net GND: no longer PROGRAMMER_PO.3, S1.P
- net N$12: no longer PROGRAMMER_PO.4
- net N$13: no longer PROGRAMMER_PO.5
- net N$8: no longer R4.1, S1.S
Other:
- moved on the sheet: BATTERY, C14, C15, C16, C17, LINEAR_REGULATOR_3.3V, PROGRAMMER_PO

Commit message: Kleine Änderungen
Connections:
- removed net N$8: MICROCHIP.!MCLR, PROGRAMMER_PO.1
- new net N$5: D1.C, R4.2
- net GND: now also PROGRAMMER_PO.3, S1.P
- net N$12: now also PROGRAMMER_PO.4
- net N$13: now also PROGRAMMER_PO.5
- net VCC: now also D1.A, MICROCHIP.!MCLR, PROGRAMMER_PO.1, R4.1, S1.S; no longer D1.C
Other:
- moved on the sheet: D1, DEBUGGING_PO, LED1, R4, R5, R6, S2

Commit message: Schematic Vollständig?
Parts:
- removed C6: 0.1uF, capacitor-wima:C2,5-3
- removed C7: 10uF, capacitor-wima:C2,5-3
Connections:
- net GND: no longer C6.2, C7.2
- net VCC: no longer C6.1, C7.1, MICROCHIP.!MCLR, MICROCHIP.AVDD, MICROCHIP.VDD, MICROCHIP.VDD_2, PROGRAMMER_PO.1, R4.1, S1.S
- net VDD33: now also MICROCHIP.!MCLR, MICROCHIP.AVDD, MICROCHIP.VDD, MICROCHIP.VDD_2, PROGRAMMER_PO.1, R4.1, S1.S
Other:
- moved on the sheet: LED2, R7

Commit message: All components placed
Parts:
- removed C13: 10uF, rcl:CPOL-EU085CS-1AR
- added C6: 0.1uF, capacitor-wima:C2,5-3
Connections:
- net GND: now also C6.2; no longer C13.-
- net VDD33: now also C6.1; no longer C13.+
Changed lines of the file:
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@@
 <part name="C10" library="capacitor-wima" library_urn="urn:adsk.eagle:library:116" deviceset="C" device="2,5-3" package3d_urn="urn:adsk.eagle:package:5436/1" value="0.1uF"/>
 <part name="C11" library="capacitor-wima" library_urn="urn:adsk.eagle:library:116" deviceset="C" device="2,5-3" package3d_urn="urn:adsk.eagle:package:5436/1" value="0.1uF"/>
-<part name="C13" library="rcl" library_urn="urn:adsk.eagle:library:334" deviceset="CPOL-EU" device="085CS-1AR" package3d_urn="urn:adsk.eagle:package:23396/3" value="10uF"/>
 <part name="GND14" library="supply1" library_urn="urn:adsk.eagle:library:371" deviceset="GND" device=""/>
 <part name="GND15" library="supply1" library_urn="urn:adsk.eagle:library:371" deviceset="GND" device=""/>
@@
 <part name="P+9" library="supply1" library_urn="urn:adsk.eagle:library:371" deviceset="VCC" device=""/>
 <part name="GND29" library="supply1" library_urn="urn:adsk.eagle:library:371" deviceset="GND" device=""/>
+<part name="C6" library="capacitor-wima" library_urn="urn:adsk.eagle:library:116" deviceset="C" device="2,5-3" package3d_urn="urn:adsk.eagle:package:5436/1" value="0.1uF"/>
 </parts>
 <sheets>
@@
 <attribute name="VALUE" x="240.284" y="43.561" size="1.778" layer="96"/>
 </instance>
-<instance part="C13" gate="G$1" x="251.46" y="48.26" smashed="yes">
-<attribute name="NAME" x="252.603" y="48.7426" size="1.778" layer="95"/>
-<attribute name="VALUE" x="252.603" y="43.6626" size="1.778" layer="96"/>
-</instance>
 <instance part="GND14" gate="1" x="226.06" y="35.56" smashed="yes">
 <attribute name="VALUE" x="223.52" y="33.02" size="1.778" layer="96"/>
@@
 <instance part="GND29" gate="1" x="-114.3" y="68.58" smashed="yes" rot="R270">
 <attribute name="VALUE" x="-116.84" y="68.58" size="1.778" layer="96" rot="R180"/>
+</instance>
+<instance part="C6" gate="G$1" x="251.46" y="48.26" smashed="yes">
+<attribute name="NAME" x="252.984" y="48.641" size="1.778" layer="95"/>
+<attribute name="VALUE" x="252.984" y="43.561" size="1.778" layer="96"/>
 </instance>
 </instances>
@@
 <wire x1="238.76" y1="38.1" x2="251.46" y2="38.1" width="0.1524" layer="91"/>
 <wire x1="251.46" y1="38.1" x2="251.46" y2="35.56" width="0.1524" layer="91"/>
-<pinref part="C13" gate="G$1" pin="-"/>
 <wire x1="251.46" y1="43.18" x2="251.46" y2="38.1" width="0.1524" layer="91"/>
 <junction x="251.46" y="38.1"/>
 <pinref part="GND15" gate="1" pin="GND"/>
+<pinref part="C6" gate="G$1" pin="2"/>
 </segment>
 <segment>
@@
 <wire x1="238.76" y1="50.8" x2="238.76" y2="55.88" width="0.1524" layer="91"/>
 <junction x="238.76" y="55.88"/>
-<pinref part="C13" gate="G$1" pin="+"/>
 <wire x1="251.46" y1="50.8" x2="251.46" y2="55.88" width="0.1524" layer="91"/>
 <junction x="251.46" y="55.88"/>
 <label x="259.08" y="55.88" size="1.778" layer="95" xref="yes"/>
-</segment>
-<segment>
+<pinref part="C6" gate="G$1" pin="1"/>
+</segment>
+<segment>

Commit message: rename ENCA and ENCB, remap PWM pins
Connections:
- removed net ENCA_A: MOTOR_L.5, MOTOR_L.6
- removed net ENCB_A: MOTOR_R.5
- removed net ENCB_B: MOTOR_R.6
- removed net MTRDRV_AI1: HBRIDGE.AIN1
- new net ENCL_A: MICROCHIP.RP21/CN26/PMA3/RC5, MOTOR_L.5
- new net ENCL_B: MICROCHIP.RP20/CN25/PMA4/RC4, MOTOR_L.6
- new net ENCR_A: MICROCHIP.RP19/CN28/PMBE/RC3, MOTOR_R.5
- new net ENCR_B: MICROCHIP.TDI/PMA9/RA9, MOTOR_R.6
- net MTRDRV_AIN1: now also HBRIDGE.AIN1
- net PWMA: now also MICROCHIP.PWM1L2/DAC1RN/RP13/CN13/PMRD/RB13; no longer MICROCHIP.PWM2L1/RP23/CN17/PMA0/RC7
- net RTS: now also MICROCHIP.PWM1L1/DAC1LN/RP15/CN11/PMCS1/RB15; no longer MICROCHIP.PWM1L2/DAC1RN/RP13/CN13/PMRD/RB13
Changed lines of the file:
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@@
 <net name="PWMA" class="0">
-<segment>
-<pinref part="MICROCHIP" gate="A" pin="PWM2L1/RP23/CN17/PMA0/RC7"/>
-<wire x1="-63.5" y1="20.32" x2="-68.58" y2="20.32" width="0.1524" layer="91"/>
-<label x="-68.58" y="20.32" size="1.778" layer="95" rot="R180" xref="yes"/>
-</segment>
 <segment>
 <pinref part="R8" gate="G$1" pin="2"/>
@@
 <label x="276.86" y="101.6" size="1.778" layer="95" xref="yes"/>
 </segment>
+<segment>
+<pinref part="MICROCHIP" gate="A" pin="PWM1L2/DAC1RN/RP13/CN13/PMRD/RB13"/>
+<wire x1="-63.5" y1="0" x2="-68.58" y2="0" width="0.1524" layer="91"/>
+<label x="-68.58" y="0" size="1.778" layer="95" rot="R180" xref="yes"/>
+</segment>
 </net>
 <net name="PWMB" class="0">
@@
 <wire x1="-35.56" y1="68.58" x2="-25.4" y2="76.2" width="0.1524" layer="91"/>
 <label x="-25.4" y="76.2" size="1.778" layer="95" xref="yes"/>
+</segment>
+<segment>
+<pinref part="HBRIDGE" gate="G$1" pin="AIN1"/>
+<wire x1="274.32" y1="96.52" x2="276.86" y2="96.52" width="0.1524" layer="91"/>
+<label x="276.86" y="96.52" size="1.778" layer="95" xref="yes"/>
 </segment>
 </net>
@@
 </segment>
 </net>
-<net name="ENCB_B" class="0">
+<net name="ENCR_B" class="0">
 <segment>
 <pinref part="MOTOR_R" gate="G$1" pin="6"/>
@@
 <label x="198.12" y="50.8" size="1.778" layer="95" xref="yes"/>
 </segment>
-</net>
-<net name="ENCB_A" class="0">
+<segment>
+<pinref part="MICROCHIP" gate="A" pin="TDI/PMA9/RA9"/>
+<wire x1="124.46" y1="2.54" x2="134.62" y2="2.54" width="0.1524" layer="91"/>
+<label x="134.62" y="2.54" size="1.778" layer="95" xref="yes"/>
+</segment>
+</net>
+<net name="ENCR_A" class="0">
 <segment>
 <pinref part="MOTOR_R" gate="G$1" pin="5"/>
@@
 <label x="172.72" y="50.8" size="1.778" layer="95" rot="R180" xref="yes"/>
 </segment>
+<segment>
+<pinref part="MICROCHIP" gate="A" pin="RP19/CN28/PMBE/RC3"/>
+<wire x1="124.46" y1="5.08" x2="134.62" y2="5.08" width="0.1524" layer="91"/>
+<label x="134.62" y="5.08" size="1.778" layer="95" xref="yes"/>
+</segment>
 </net>
 <net name="BO1" class="0">
@@
 </segment>
 <segment>
-<pinref part="MICROCHIP" gate="A" pin="PWM1L2/DAC1RN/RP13/CN13/PMRD/RB13"/>
-<wire x1="-63.5" y1="0" x2="-68.58" y2="0" width="0.1524" layer="91"/>
-<label x="-68.58" y="0" size="1.778" layer="95" rot="R180" xref="yes"/>
+<pinref part="MICROCHIP" gate="A" pin="PWM1L1/DAC1LN/RP15/CN11/PMCS1/RB15"/>
+<wire x1="-63.5" y1="-10.16" x2="-68.58" y2="-10.16" width="0.1524" layer="91"/>
+<label x="-68.58" y="-10.16" size="1.778" layer="95"/>
+<label x="-68.58" y="-10.16" size="1.778" layer="95" rot="R180" xref="yes"/>
 </segment>
 </net>
@@
 </segment>
 </net>
-<net name="MTRDRV_AI1" class="0">
-<segment>
-<pinref part="HBRIDGE" gate="G$1" pin="AIN1"/>
-<wire x1="274.32" y1="96.52" x2="276.86" y2="96.52" width="0.1524" layer="91"/>
-<label x="276.86" y="96.52" size="1.778" layer="95" xref="yes"/>
-</segment>
-</net>
 <net name="B01" class="0">
 <segment>
@@
 </segment>
 </net>
-<net name="ENCA_A" class="0">
+<net name="ENCL_B" class="0">
+<segment>
+<pinref part="MOTOR_L" gate="G$1" pin="6"/>
+<wire x1="195.58" y1="27.94" x2="198.12" y2="25.4" width="0.1524" layer="91"/>
+<label x="198.12" y="25.4" size="1.778" layer="95" xref="yes"/>
+</segment>
+<segment>
+<pinref part="MICROCHIP" gate="A" pin="RP20/CN25/PMA4/RC4"/>
+<wire x1="124.46" y1="7.62" x2="134.62" y2="7.62" width="0.1524" layer="91"/>
+<label x="134.62" y="7.62" size="1.778" layer="95" xref="yes"/>
+</segment>
+</net>
+<net name="N$3" class="0">
+<segment>
+<pinref part="Y1" gate="G$1" pin="X1"/>
+<pinref part="C2" gate="G$1" pin="1"/>
+</segment>
+</net>
+<net name="N$4" class="0">
+<segment>
+<pinref part="Y1" gate="G$1" pin="X2"/>
+<pinref part="C3" gate="G$1" pin="2"/>
+</segment>
+</net>
+<net name="N$5" class="0">
+<segment>
+<pinref part="D1" gate="1" pin="C"/>
+<pinref part="R4" gate="G$1" pin="2"/>
+<wire x1="-149.86" y1="-53.34" x2="-144.78" y2="-53.34" width="0.1524" layer="91"/>
+</segment>
+</net>
+<net name="ENCL_A" class="0">
 <segment>
 <pinref part="MOTOR_L" gate="G$1" pin="5"/>
@@
 </segment>
 <segment>
-<pinref part="MOTOR_L" gate="G$1" pin="6"/>
-<wire x1="195.58" y1="27.94" x2="198.12" y2="25.4" width="0.1524" layer="91"/>
-<label x="198.12" y="25.4" size="1.778" layer="95" xref="yes"/>
-</segment>
-</net>
-<net name="N$3" class="0">
-<segment>
-<pinref part="Y1" gate="G$1" pin="X1"/>
-<pinref part="C2" gate="G$1" pin="1"/>
-</segment>
-</net>
-<net name="N$4" class="0">
-<segment>
-<pinref part="Y1" gate="G$1" pin="X2"/>
-<pinref part="C3" gate="G$1" pin="2"/>
-</segment>
-</net>
-<net name="N$5" class="0">
-<segment>
-<pinref part="D1" gate="1" pin="C"/>
-<pinref part="R4" gate="G$1" pin="2"/>
-<wire x1="-149.86" y1="-53.34" x2="-144.78" y2="-53.34" width="0.1524" layer="91"/>
-</segment>
-</net>
+<pinref part="MICROCHIP" gate="A" pin="RP21/CN26/PMA3/RC5"/>
+<wire x1="124.46" y1="10.16" x2="134.62" y2="10.16" width="0.1524" layer="91"/>
+<label x="134.62" y="10.16" size="1.778" layer="95" xref="yes"/>
+</segment>
+</net>
