File: project.sch (EAGLE design)
At the start: 42 parts, among them Y1 ABM8-20.000MHZ-B2-T

Commit message: add 5V voltage regulator
Parts:
- added C12, C7: 1uF, capacitor-wima:C2,5-3
- added C13, C19, C20: 100nF, capacitor-wima:C2,5-3
- added LINEAR_REGULATOR_5V: ADP3338AKCZ-5-R7, ADP3338AKCZ-5-R7:ADP3338AKCZ-5-R7
Connections:
- removed net N$27: DEBUGGING_PO.10
- new net 5V: C13.1, C14.1, C19.1, C20.1, C7.1, JP1(GP2Y0A51SK0F).1, JP2(GP2Y0A51SK0F).1, JP3(GP2Y0A51SK0F).1, LINEAR_REGULATOR_3.3V.INPUT, LINEAR_REGULATOR_5V.OUT
- net GND: now also C12.2, C13.2, C19.2, C20.2, C7.2, DEBUGGING_PO.10, LINEAR_REGULATOR_5V.GND
- net VCC: no longer JP1(GP2Y0A51SK0F).1, JP2(GP2Y0A51SK0F).1, JP3(GP2Y0A51SK0F).1
- net VM: now also C12.1, LINEAR_REGULATOR_5V.IN; no longer C14.1, LINEAR_REGULATOR_3.3V.INPUT
Other:
- moved on the sheet: BATTERY

Commit message: Leds added, 5v Regulator Moved, Bluetooth removed
Parts:
- removed BLUETOOTH_UART: (no value), pinhead:PINHD-1X6
- added LED4, LED5: TLLG4400, led:TLLG4400
- added R10, R9: 10k, rcl:R-EU_0204/2V
Connections:
- new net LED2: R7.2
- new net LED3: R8.2
- new net LED4: R9.2
- new net LED5: R10.2
- new net N$6: LED4.A, R9.1
- new net N$8: LED5.A, R10.1
- net 5V: no longer C14.1, LINEAR_REGULATOR_3.3V.INPUT
- net CTS: no longer BLUETOOTH_UART.6
- net GND: now also LED4.C, LED5.C; no longer BLUETOOTH_UART.2
- net PWMA: no longer R8.2
- net PWMB: no longer R7.2
- net RTS: no longer BLUETOOTH_UART.3
- net RX: no longer BLUETOOTH_UART.4
- net TX: no longer BLUETOOTH_UART.5
- net VDD33: no longer BLUETOOTH_UART.1
- net VM: now also C14.1, LINEAR_REGULATOR_3.3V.INPUT
Other:
- moved on the sheet: BATTERY, C12, C14, C15, C16, C17, C7, LINEAR_REGULATOR_3.3V, LINEAR_REGULATOR_5V

Commit message: Small Changes
Connections:
- net RTS renamed PMW_L
- removed net CTS: MICROCHIP.PWM1H2/DAC1RP/RP12/CN14/PMD0/RB12
- removed net N$12: MICROCHIP.PGEC1/AN3/C2IN+/RP1/CN5/RB1, PROGRAMMER_PO.4
- removed net N$13: MICROCHIP.PGED1/AN2/C2IN-/RP0/CN4/RB0, PROGRAMMER_PO.5
- removed net N$15: MICROCHIP.PWM2H1/RP22/CN18/PMA1/RC6, R6.2
- removed net RX: MICROCHIP.PGEC2/PWM1L3/RP11/CN15/PMD1/RB11
- removed net TX: MICROCHIP.PGED2/EMCD2/PWM1H3/RP10/CN16/PMD2/RB10
- new net 3.3V: C10.1, C11.1, C15.1, C16.1, C17.1, C6.1, D1.A, HBRIDGE.VCC, LINEAR_REGULATOR_3.3V.OUTPUT, MOTOR_L.4, MOTOR_R.4, PROGRAMMER_PO.2
- new net PGC1: PROGRAMMER_PO.5
- new net PGD1: PROGRAMMER_PO.4
- new net PGEC1: MICROCHIP.PGEC1/AN3/C2IN+/RP1/CN5/RB1
- new net PGED1: MICROCHIP.PGED1/AN2/C2IN-/RP0/CN4/RB0
- new net PMW_R: MICROCHIP.PWM1L2/DAC1RN/RP13/CN13/PMRD/RB13
- net PWMA: no longer MICROCHIP.PWM1L2/DAC1RN/RP13/CN13/PMRD/RB13
- net PWMB: no longer MICROCHIP.PWM1H1/DAC1LP/RTCC/RP14/CN12/PMWR/RB14
- net STBY: no longer MICROCHIP.SDA1/RP9/CN21/PMD3/RB9
- net VCC: no longer C15.1, C16.1, C17.1, D1.A, HBRIDGE.VCC, LINEAR_REGULATOR_3.3V.OUTPUT, PROGRAMMER_PO.2
- net VDD33: no longer C10.1, C11.1, C6.1, MOTOR_L.4, MOTOR_R.4

Commit message: Added Bluetooth Module
Parts:
- removed LED5: TLLG4400, led:TLLG4400
- removed R10, R6: 10k, rcl:R-EU_0204/2V
- added BLUETOOTH: RN4871-I_RM130, RN4871-I_RM130:RN4871-I_RM130
- added C21: 100nF, capacitor-wima:C2,5-3
- added C22: 0.1uF, capacitor-wima:C2,5-3
- added C23: 10uF, capacitor-wima:C2,5-3
- C10, C11, C6: value 0.1uF -> 100nF
Connections:
- net PWMB renamed PWM_R
- removed net LED5: R10.2
- removed net N$16 (its old number): LED1.A, R6.1
- removed net PGC1: PROGRAMMER_PO.5
- removed net PGD1: PROGRAMMER_PO.4
- removed net PWMA: DEBUGGING_PO.1, HBRIDGE.PWMA
- removed net VCC: S2.S
- removed net VDD33: MICROCHIP.!MCLR, MICROCHIP.AVDD, MICROCHIP.VDD, MICROCHIP.VDD_2, PROGRAMMER_PO.1, R4.1, S1.S
- new net N$12: LED1.A, R4.1, S1.S
- new net N$13: C21.2, MICROCHIP.!MCLR
- new net N$14: C11.1, MICROCHIP.VDD_2
- new net N$15: C10.1, MICROCHIP.VDD
- new net N$20: BLUETOOTH.P1_2
- new net N$21: BLUETOOTH.P1_3
- new net N$22: BLUETOOTH.P1_7
- new net N$23: BLUETOOTH.P1_6
- new net N$24: BLUETOOTH.P3_6
- new net N$25: BLUETOOTH.RST_N
- new net N$26: BLUETOOTH.P0_0
- new net N$27: BLUETOOTH.P0_2
- new net N$31: BLUETOOTH.P2_7
- new net N$32: BLUETOOTH.P2_0
- new net N$9: C21.1, LED1.C, PROGRAMMER_PO.1
- new net PWM_L: HBRIDGE.PWMA
- new net RX: BLUETOOTH.UART_RX
- new net TX: BLUETOOTH.UART_TX
- net 3.3V: now also BLUETOOTH.VBAT, C10.2, C11.2, S2.S; no longer C10.1, C11.1
- net 5V: now also C22.1, C23.1, HBRIDGE.STBY
- net ENCL_A: now also MICROCHIP.PWM2H1/RP22/CN18/PMA1/RC6; no longer MICROCHIP.RP21/CN26/PMA3/RC5
- net ENCL_B: now also MICROCHIP.SDA1/RP9/CN21/PMD3/RB9; no longer MICROCHIP.RP20/CN25/PMA4/RC4
- net ENCR_A: now also MICROCHIP.PWM2L1/RP23/CN17/PMA0/RC7; no longer MICROCHIP.RP19/CN28/PMBE/RC3
- net ENCR_B: now also MICROCHIP.RP24/CN20/PMA5/RC8; no longer MICROCHIP.TDI/PMA9/RA9
- net GND: now also BLUETOOTH.GND_1, BLUETOOTH.GND_2, C22.2, C23.2; no longer C10.2, C11.2, C6.2, LED1.C, LED5.C
- net LED2: now also MICROCHIP.PGED2/EMCD2/PWM1H3/RP10/CN16/PMD2/RB10
- net LED3: now also MICROCHIP.PGEC2/PWM1L3/RP11/CN15/PMD1/RB11
- net LED4: now also MICROCHIP.PWM1H2/DAC1RP/RP12/CN14/PMD0/RB12
- net N$8: now also C6.2, MICROCHIP.AVDD; no longer LED5.A, R10.1
- net PGEC1: now also PROGRAMMER_PO.5
- net PGED1: now also PROGRAMMER_PO.4
- net PMW_L: now also DEBUGGING_PO.1
- net STBY: no longer HBRIDGE.STBY
Other:
- moved on the sheet: BATTERY, C1, C10, C11, C12, C13, C14, C15, C16, C17, C18, C19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

Commit message: group and place components in board
Parts:
- added C24, C25, C26, C27: 100nF, capacitor-wima:C2,5-3
- C8: value 0.1uF -> 10uF
Connections:
- removed net LED3: MICROCHIP.PGEC2/PWM1L3/RP11/CN15/PMD1/RB11, R8.2
- removed net LED4: MICROCHIP.PWM1H2/DAC1RP/RP12/CN14/PMD0/RB12, R9.2
- removed net N$14: C11.1, MICROCHIP.VDD_2
- removed net N$15: C10.1, MICROCHIP.VDD
- removed net N$8: C6.2, MICROCHIP.AVDD
- removed net STBY: DEBUGGING_PO.5
- net 3.3V: now also C24.1, C25.1, C26.1, C27.1, MICROCHIP.AVDD, MICROCHIP.VDD, MICROCHIP.VDD_2
- net GND: now also C10.1, C11.1, C24.2, C25.2, C26.2, C27.2, C6.2
- net PWM_L: now also R8.2
- net PWM_R: now also R9.2
- net RX: now also MICROCHIP.RP21/CN26/PMA3/RC5
- net TX: now also MICROCHIP.RP20/CN25/PMA4/RC4
Other:
- moved on the sheet: C10, C11, C6

Commit message: route board
Connections:
- removed net B01: HBRIDGE.BO1_2
- removed net PMW_L: DEBUGGING_PO.1, MICROCHIP.PWM1L1/DAC1LN/RP15/CN11/PMCS1/RB15
- removed net PMW_R: MICROCHIP.PWM1L2/DAC1RN/RP13/CN13/PMRD/RB13
- net AN0: now also MICROCHIP.AN1/VREF-/CN3/RA1; no longer MICROCHIP.AN0/VREF+/CN2/RA0
- net AN1: now also MICROCHIP.AN0/VREF+/CN2/RA0; no longer MICROCHIP.AN1/VREF-/CN3/RA1
- net BO1: now also HBRIDGE.BO1_1, HBRIDGE.BO1_2
- net ENCL_A: now also MICROCHIP.SDA1/RP9/CN21/PMD3/RB9; no longer MICROCHIP.PWM2H1/RP22/CN18/PMA1/RC6
- net ENCL_B: now also MICROCHIP.PWM2H1/RP22/CN18/PMA1/RC6; no longer MICROCHIP.SDA1/RP9/CN21/PMD3/RB9
- net N$16: now also MICROCHIP.TMS/PMA10/RA10; no longer MICROCHIP.INT0/RP7/CN23/PMD5/RB7
- net PGEC1: now also MICROCHIP.PGEC2/PWM1L3/RP11/CN15/PMD1/RB11; no longer MICROCHIP.PGEC1/AN3/C2IN+/RP1/CN5/RB1
- net PGED1: now also MICROCHIP.PWM1H2/DAC1RP/RP12/CN14/PMD0/RB12; no longer MICROCHIP.PGED1/AN2/C2IN-/RP0/CN4/RB0
- net PWM_L: now also MICROCHIP.PWM1L1/DAC1LN/RP15/CN11/PMCS1/RB15
- net PWM_R: now also MICROCHIP.PWM1L2/DAC1RN/RP13/CN13/PMRD/RB13; no longer DEBUGGING_PO.3
- net RX: now also MICROCHIP.SCL1/RP8/CN22/PMD4/RB8; no longer MICROCHIP.RP21/CN26/PMA3/RC5
- net TX: now also MICROCHIP.INT0/RP7/CN23/PMD5/RB7; no longer MICROCHIP.RP20/CN25/PMA4/RC4
Other:
- moved on the sheet: R5, S2

Commit message: Progress!
Parts:
- removed BATTERY: (no value), pinhead:PINHD-1X2
- removed C12, C7: 1uF, capacitor-wima:C2,5-3
- removed LINEAR_REGULATOR_5V: ADP3338AKCZ-5-R7, ADP3338AKCZ-5-R7:ADP3338AKCZ-5-R7
- added C29, C30, C31: C0805J104K1RACAUTO, C0805J104K1RACAUTO:C0805J104K1RACAUTO
- added IC1: ADP3338AKCZ-5-R7, ADP3338AKCZ-5-R7:ADP3338AKCZ-5-R7
- added J1: 22-23-2021, 22-23-2021:22-23-2021
- added R10, R6: 4.7k, rcl:R-EU_0204/2V
- LED1, LED2, LED3, LED4: value TLLG4400 -> APT3216LSECK_J3-PRV; device led:TLLG4400 -> APT3216LSECK_J3-PRV:APT3216LSECK_J3-PRV
- R1: value 10k -> 4.7k
- S1, S2: value TL32PO -> B3F-1020; device switch:TL32PO -> B3F-1020:B3F-1020
Connections:
- net N$24 renamed RTS
- net N$26 renamed CTS
- net 3.3V: now also R10.2, R6.2, S2.3; no longer S2.S
- net 5V: now also C29.1, IC1.OUT; no longer C7.1, LINEAR_REGULATOR_5V.OUT
- net GND: now also C29.2, C30.2, C31.2, IC1.GND, J1.2, LED2.K, LED3.K, LED4.K, S1.4; no longer BATTERY.2, C12.2, C7.2, LED2.C, LED3.C, LED4.C, LINEAR_REGULATOR_5V.GND, S1.P
- net N$12: now also S1.1; no longer S1.S
- net N$16: now also S2.2; no longer S2.P
- net N$25: now also C31.1, R10.1
- net N$27: now also R6.1
- net N$9: now also LED1.K; no longer LED1.C
- net PGEC1: now also MICROCHIP.PGEC1/AN3/C2IN+/RP1/CN5/RB1
- net PGED1: now also MICROCHIP.PGED1/AN2/C2IN-/RP0/CN4/RB0
- net VM: now also C30.1, IC1.IN, J1.1; no longer BATTERY.1, C12.1, LINEAR_REGULATOR_5V.IN
Other:
- moved on the sheet: BLUETOOTH, C27, LED1, LED2, LED3, LED4, R7, R8, R9

Commit message: Progress!
Parts:
- removed C10, C11, C13, C16, C17, C19, C20, C21, C24, C25, C26, C27, C4, C5, C6: 100nF, capacitor-wima:C2,5-3
- removed C15: 0.1µF, capacitor-wima:C2,5-3
- removed C22: 0.1uF, capacitor-wima:C2,5-3
- added C12, C7: 0805YC106KAT2A, 0805YC106KAT2A:0805YC106KAT2A
- added C28, C32, C33, C34, C35, C36, C37, C38, C39, C40, C41, C42, C43, C44, C46: C0805J104K1RACAUTO, C0805J104K1RACAUTO:C0805J104K1RACAUTO
- C1: value 100nF -> C0805J104K1RACAUTO; device capacitor-wima:C2,5-3 -> C0805J104K1RACAUTO:C0805J104K1RACAUTO
- C14: value 0.33µF -> C0805J104K1RACAUTO; device capacitor-wima:C2,5-3 -> C0805J104K1RACAUTO:C0805J104K1RACAUTO
- C23: value 10uF -> C0805J104K1RACAUTO; device capacitor-wima:C2,5-3 -> C0805J104K1RACAUTO:C0805J104K1RACAUTO
- C30: value C0805J104K1RACAUTO -> 1µF
- C8: value 10uF -> 0805YC106KAT2A; device capacitor-wima:C2,5-3 -> 0805YC106KAT2A:0805YC106KAT2A
- C9: value 10uF -> 08053C334KAZ2A; device capacitor-wima:C2,5-3 -> 08053C334KAZ2A:08053C334KAZ2A
Connections:
- net 3.3V: now also C1.1, C14.1, C23.1, C28.1, C38.1, C39.1, C40.1, C42.1, C43.1, C44.1; no longer C10.2, C11.2, C15.1, C16.1, C17.1, C24.1, C25.1, C26.1, C27.1, C6.1
- net 5V: now also C35.1, C36.1, C37.1, C46.1, C8.1; no longer C13.1, C19.1, C20.1, C22.1, C23.1
- net AN0: now also C32.1; no longer C1.1
- net AN1: now also C33.1; no longer C4.1
- net AN4: now also C34.1; no longer C5.1
- net GND: now also C12.2, C28.2, C32.2, C33.2, C34.2, C35.2, C36.2, C37.2, C38.2, C39.2, C40.2, C42.2, C43.2, C44.2, C46.2, C7.2; no longer C10.1, C11.1, C13.2, C15.2, C16.2, C17.2, C19.2, C20.2, C22.2, C24.2, C25.2, C26.2, C27.2, C4.2, C5.2, C6.2
- net N$13: now also C41.2; no longer C21.2
- net N$9: now also C41.1; no longer C21.1
- net VM: now also C12.1, C7.1; no longer C14.1, C8.1
