File: project.brd (EAGLE design)
At the start: 160 x 100 mm, 58 parts, among them IC1 ADP3338AKCZ-5-R7, J1 22-23-2021, Y1 ABM8-20.000MHZ-B2-T

Commit message: Saving Progress
Parts:
- moved R13 202.0 mm to (41.9, 49.5)
- moved R14 201.5 mm to (40.6, 43.2), turned to 90 degrees
- moved R11 169.0 mm to (29.2, 24.1)
- moved R12 169.0 mm to (26.7, 20.3)
- moved R4 169.0 mm to (5.08, 14.0)
- moved R5 169.0 mm to (19.1, 7.62)
- moved C31 72.8 mm to (41.9, 47.0)
- moved C32 66.5 mm to (35.6, 10.2)
- moved C33 66.5 mm to (29.2, 7.62)
- moved C34 66.5 mm to (22.9, 5.08)
- moved C1 1.80 mm to (33.0, 52.1), turned to 90 degrees
- moved C42 1.27 mm to (64.8, 58.4)
- moved D1 1.27 mm to (77.5, 45.7)
Routing:
- net 3.3V: track 157.7 -> 175.7 mm
- net N$25: track 0.00 -> 7.65 mm
