File: project.brd (EAGLE design)
At the start: 160 x 100 mm, 58 parts, among them IC1 ADP3338AKCZ-5-R7, J1 22-23-2021, Y1 ABM8-20.000MHZ-B2-T

Commit message: progress
Parts:
- moved R4 273.4 mm to (97.6, 62.4), turned to 180 degrees
- moved R5 263.3 mm to (99.9, 56.2), turned to 180 degrees
- moved R11 250.0 mm to (96.6, 69.1), turned to 180 degrees
- moved R12 232.9 mm to (91.4, 34.3)
- moved R14 208.8 mm to (43.2, 52.1)
- moved R13 199.4 mm to (36.8, 52.1)
- moved C34 161.9 mm to (103.7, 56.3)
- moved C33 156.8 mm to (101.9, 62.5)
- moved C32 153.2 mm to (101.1, 69.3)
- moved C31 71.1 mm to (39.4, 47.0), turned to 90 degrees
- moved Y1 21.7 mm to (52.1, 54.6)
- moved C2 19.2 mm to (48.3, 52.1), turned to 90 degrees
- moved C41 17.7 mm to (80.9, 41.3)
- moved C3 16.1 mm to (52.1, 52.1), turned to 0 degrees
- moved C40 8.52 mm to (48.3, 55.9), turned to 270 degrees
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Connections:
- net AN0: now also C33.1, JP2(GP2Y0A51SK0F).2, R4.1; no longer C32.1, JP1(GP2Y0A51SK0F).2, R11.1
- net AN1: now also C34.1, JP3(GP2Y0A51SK0F).2, R5.1; no longer C33.1, JP2(GP2Y0A51SK0F).2, R4.1
- net AN4: now also C32.1, JP1(GP2Y0A51SK0F).2, R11.1; no longer C34.1, JP3(GP2Y0A51SK0F).2, R5.1
- net ENCL_A: now also MICROCHIP.36; no longer MICROCHIP.1
- net ENCL_B: now also MICROCHIP.35; no longer MICROCHIP.2
- net ENCR_A: now also MICROCHIP.37; no longer MICROCHIP.3
- net ENCR_B: now also MICROCHIP.38; no longer MICROCHIP.4
- net STBY: now also MICROCHIP.13
Routing:
- net AN4: track 0.00 -> 54.7 mm, vias 0 -> 2
- net AN1: track 0.00 -> 53.0 mm, vias 0 -> 2
- net AN0: track 0.00 -> 51.9 mm, vias 0 -> 2
- net PWM_L: track 0.00 -> 37.5 mm, vias 0 -> 4
- net N$16: track 0.00 -> 36.2 mm
- net ENCL_A: track 0.00 -> 33.7 mm, vias 0 -> 2
- net STBY: track 0.00 -> 32.3 mm, vias 0 -> 4
- net 3.3V: track 157.7 -> 188.4 mm
- net ENCR_A: track 0.00 -> 29.8 mm, vias 0 -> 2
- net ENCL_B: track 0.00 -> 28.4 mm, vias 0 -> 2
- net ENCR_B: track 0.00 -> 28.2 mm, vias 0 -> 2
- net PGEC1: track 0.00 -> 28.1 mm, vias 0 -> 4
- net PGED1: track 0.00 -> 27.2 mm, vias 0 -> 4
- net PWM_R: track 0.00 -> 25.5 mm, vias 0 -> 2
- net N$13: track 2.66 -> 23.3 mm, vias 0 -> 4
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Other:
- board size 160 x 100 mm -> 88.9 x 75.7 mm
